Commit message: some bug fixes

File: urdf/awl_description.xacro (robot description, xacro)
@@ -48,5 +48,5 @@
     <visual>
       <geometry>
-        <mesh filename="package://awl_description/meshes/main_wheel.dae" scale="1 1 1" />
+        <mesh filename="package://luci_third_party/meshes/main_wheel.dae" scale="1 1 1" />
       </geometry>
     </visual>
@@ -70,5 +70,5 @@
     <visual>
       <geometry>
-        <mesh filename="package://awl_description/meshes/main_wheel.dae" scale="1 1 1" />
+        <mesh filename="package://luci_third_party/meshes/main_wheel.dae" scale="1 1 1" />
       </geometry>
     </visual>
@@ -94,5 +94,5 @@
     <visual>
       <geometry>
-        <mesh filename="package://awl_description/meshes/caster_wheels.dae" scale="1 1 1" />
+        <mesh filename="package://luci_third_party/meshes/caster_wheels.dae" scale="1 1 1" />
       </geometry>
     </visual>
@@ -125,5 +125,5 @@
     <visual>
       <geometry>
-        <mesh filename="package://awl_description/meshes/caster_wheels.dae" scale="1 1 1" />
+        <mesh filename="package://luci_third_party/meshes/caster_wheels.dae" scale="1 1 1" />
       </geometry>
     </visual>
@@ -157,5 +157,5 @@
     <visual>
       <geometry>
-        <mesh filename="package://awl_description/meshes/caster_wheels.dae" scale="1 1 1" />
+        <mesh filename="package://luci_third_party/meshes/caster_wheels.dae" scale="1 1 1" />
       </geometry>
     </visual>
@@ -188,5 +188,5 @@
     <visual>
       <geometry>
-        <mesh filename="package://awl_description/meshes/caster_wheels.dae" scale="1 1 1" />
+        <mesh filename="package://luci_third_party/meshes/caster_wheels.dae" scale="1 1 1" />
       </geometry>
     </visual>
